Commit message: ★ 스캔 머지 추가 및 파라미터 수정

File: tetraDS_description/urdf/tetraDS/tetraDS.xacro (robot description, xacro)
@@ -46,4 +46,18 @@
     <child link="laser_link2" />
   </joint>
+  <link name="laser_merge">
+      <visual>
+        <origin xyz="0 0 0" rpy="0 0 0" />
+        <geometry>
+          <box size="0.01 0.01 0.01" />
+        </geometry>
+        <material name="Grey" />
+      </visual>
+  </link>
+  <joint name="base_link_to_laser_merge" type="fixed">
+    <origin xyz="0.0 0.0 0.15182" rpy="0 0 0" />
+    <parent link="base_link"/>
+    <child link="laser_merge" />
+  </joint>
   <link name="imu_link">
       <visual>
@@ -70,5 +84,5 @@
   </link>
   <joint name="usb_cam" type="fixed">
-    <origin xyz="0.3325 0.0 0.156" rpy="1.5708 3.14159 1.5708"/>
+    <origin xyz="0.3325 0.0 0.156" rpy="${PI*0.5} ${PI} ${PI*0.5}"/>
     <parent link="base_link"/>
     <child link="usb_cam" />
@@ -87,4 +101,18 @@
     <parent link="base_link"/>
     <child link="Front_bumper" />
+  </joint>
+ <link name="Rear_bumper">
+      <visual>
+        <origin xyz="0 0 0" rpy="0 0 0" />
+        <geometry>
+          <box size="0.01 0.580 0.01" />
+        </geometry>
+        <material name="TransparentBlack" />
+      </visual>
+  </link>
+  <joint name="Rear_bumper" type="fixed">
+    <origin xyz="-0.434 0.0 -0.05" rpy="0 0 3.14" />
+    <parent link="base_link"/>
+    <child link="Rear_bumper" />
   </joint>
  <link name="camera1_link">

Commit message: ♥ 레이저 필터 추가 및 뎁스카메라로 도킹하게 변경

File: tetraDS_description/urdf/tetraDS/tetraDS.xacro (robot description, xacro)
@@ -126,5 +126,5 @@
   </link>
   <joint name="camera1_link" type="fixed">
-    <origin xyz="0.39660 0 0.095" rpy="0 0 0" />
+    <origin xyz="0.39660 0.05 0.095" rpy="0 0 0" />
     <parent link="base_link"/>
     <child link="camera1_link" />

Commit message: ★ h모델 도킹시 보정 로직 추가

File: tetraDS_description/urdf/tetraDS/tetraDS.xacro (robot description, xacro)
@@ -84,5 +84,5 @@
   </link>
   <joint name="usb_cam" type="fixed">
-    <origin xyz="0.3325 0.0 0.156" rpy="${PI*0.5} ${PI} ${PI*0.5}"/>
+    <origin xyz="0.3325 -0.06 0.156" rpy="${PI*0.5} ${PI} ${PI*0.5}"/>
     <parent link="base_link"/>
     <child link="usb_cam" />
@@ -126,5 +126,5 @@
   </link>
   <joint name="camera1_link" type="fixed">
-    <origin xyz="0.39660 0.05 0.095" rpy="0 0 0" />
+    <origin xyz="0.39660 0.0 0.095" rpy="0 0 0" />
     <parent link="base_link"/>
     <child link="camera1_link" />
